File: acker_pcb/Rlaarlo_PDB/Rlaarlo_PDB.kicad_sch (KiCad schematic)
At the start: 0 parts

Commit message: initial schematic
Parts:
- added Buck1: xl4016, symbol buck_module:buck_module
- added Buck2: xl4015, symbol buck_module:buck_module
- added J1: xt 60, symbol Connector:Conn_01x02_Pin
- added J2: Conn_01x03_Pin, symbol Connector:Conn_01x03_Pin
- added J3: Conn_01x02_Pin, symbol Connector:Conn_01x02_Pin
- added SW1, SW2, SW3: SW_SPST, symbol Switch:SW_SPST
- added vesc1: (no value), symbol vesc:vesc
Connections:
- new net: Buck2.3 (v_out_+), J2.1 (Pin_1), vesc1.3 (servo+)
- new net: J2.3 (Pin_3), vesc1.5 (pwm)
- new net: Buck1.1 (v_in_+), SW3.2 (B)
- new net: SW1.2 (B), vesc1.1 (v+)
- new net: Buck1.3 (v_out_+), J3.2 (Pin_2)
- new net: Buck2.1 (v_in_+), SW2.2 (B)
- new net +15V: J1.2 (Pin_2), SW1.1 (A), SW2.1 (A), SW3.1 (A)
- new net GND: Buck1.2 (v_in_-), Buck1.4 (v_out_-), Buck2.2 (v_in_-), Buck2.4 (v_out_-), J1.1 (Pin_1), J2.2 (Pin_2), J3.1 (Pin_1), vesc1.2 (v-), vesc1.4 (servo-)

Commit message: updates for footprint
Parts:
- Buck1: footprint (none) -> acker:XL4016 BUCK
- Buck2: footprint (none) -> acker:XL4015 Buck
- J1: footprint (none) -> Connector_AMASS:AMASS_XT60-M_1x02_P7.20mm_Vertical
- J2: footprint (none) -> Connector_PinHeader_2.54mm:PinHeader_1x03_P2.54mm_Horizontal
- J3: footprint (none) -> Connector_PinHeader_2.54mm:PinHeader_1x02_P2.54mm_Horizontal
- SW1, SW2, SW3: footprint (none) -> acker:spst_switch
Connections:
- net at Buck2.3 (v_out_+), J2.1 (Pin_1): no longer vesc1.3 (servo+)
- no-connect marks 0 -> 1
Changed lines of the file:
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@@
-	)
-	(junction
-		(at 104.14 50.8)
-		(diameter 0)
-		(color 0 0 0 0)
 	)
 	(junction
@@
 		(color 0 0 0 0)
 	)
+	(no_connect
+		(at 96.52 50.8)
+	)
 	(wire
 		(pts
@@
 	(wire
 		(pts
-			(xy 104.14 66.04) (xy 104.14 50.8)
-		)
-		(stroke
-			(width 0)
-			(type default)
-		)
-	)
-	(wire
-		(pts
 			(xy 29.21 87.63) (xy 35.56 87.63)
 		)
@@
 	(wire
 		(pts
-			(xy 96.52 50.8) (xy 104.14 50.8)
-		)
-		(stroke
-			(width 0)
-			(type default)
-		)
-	)
-	(wire
-		(pts
 			(xy 36.83 90.17) (xy 48.26 90.17)
 		)
@@
 	(wire
 		(pts
-			(xy 104.14 50.8) (xy 104.14 34.29)
+			(xy 104.14 34.29) (xy 104.14 66.04)
 		)
 		(stroke
@@
 			)
 		)
-		(property "Footprint" ""
+		(property "Footprint" "Connector_PinHeader_2.54mm:PinHeader_1x03_P2.54mm_Horizontal"
 			(at 113.03 31.75 0)
 			(hide yes)
@@
 			)
 		)
-		(property "Footprint" ""
+		(property "Footprint" "acker:spst_switch"
 			(at 59.69 80.01 0)
 			(hide yes)
@@
 			)
 		)
-		(property "Footprint" ""
+		(property "Footprint" "acker:spst_switch"
 			(at 62.23 50.8 0)
 			(hide yes)
@@
 			)
 		)
-		(property "Footprint" ""
+		(property "Footprint" "Connector_AMASS:AMASS_XT60-M_1x02_P7.20mm_Vertical"
 			(at 53.34 90.17 0)
 			(hide yes)
@@
 			)
 		)
-		(property "Footprint" ""
+		(property "Footprint" "Connector_PinHeader_2.54mm:PinHeader_1x02_P2.54mm_Horizontal"
 			(at 125.73 82.55 0)
 			(hide yes)
@@
 			)
 		)
-		(property "Footprint" ""
+		(property "Footprint" "acker:spst_switch"
 			(at 59.69 66.04 0)
 			(hide yes)
@@
 			)
 		)
-		(property "Footprint" ""
+		(property "Footprint" "acker:XL4016 BUCK"
 			(at 80.01 81.28 0)
 			(hide yes)
@@
 			)
 		)
-		(property "Footprint" ""
+		(property "Footprint" "acker:XL4015 Buck"
 			(at 80.01 67.31 0)
 			(hide yes)

Commit message: lenevo work
Parts:
- vesc1: footprint (none) -> acker:vesc
Changed lines of the file:
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@@
 			)
 		)
-		(property "Footprint" ""
+		(property "Footprint" "acker:vesc"
 			(at 85.09 48.26 0)
 			(hide yes)

Commit message: pcb design updates
Parts:
- J3: footprint Connector_PinHeader_2.54mm:PinHeader_1x02_P2.54mm_Horizontal -> TerminalBlock:TerminalBlock_MaiXu_MX126-5.0-02P_1x02_P5.00mm
Connections:
- net GND: now also J2.1 (Pin_1), vesc1.1 (v-), vesc1.3 (servo-); no longer J2.2 (Pin_2), vesc1.2 (v-), vesc1.4 (servo-)
- net at Buck2.3 (v_out_+): now also J2.2 (Pin_2); no longer J2.1 (Pin_1)
- net at SW1.2 (B): now also vesc1.2 (v+); no longer vesc1.1 (v+)
Changed lines of the file:
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@@
 	)
 	(no_connect
-		(at 96.52 50.8)
+		(at 96.52 48.26)
 	)
 	(wire
@@
 	(wire
 		(pts
+			(xy 96.52 50.8) (xy 99.06 50.8)
+		)
+		(stroke
+			(width 0)
+			(type default)
+		)
+	)
+	(wire
+		(pts
 			(xy 105.41 71.12) (xy 105.41 68.58)
 		)
@@
 	(wire
 		(pts
-			(xy 96.52 48.26) (xy 100.33 48.26)
-		)
-		(stroke
-			(width 0)
-			(type default)
-		)
-	)
-	(wire
-		(pts
 			(xy 48.26 80.01) (xy 54.61 80.01)
 		)
@@
 	(wire
 		(pts
+			(xy 104.14 31.75) (xy 107.95 31.75)
+		)
+		(stroke
+			(width 0)
+			(type default)
+		)
+	)
+	(wire
+		(pts
 			(xy 69.85 45.72) (xy 69.85 39.37)
 		)
@@
 	(wire
 		(pts
-			(xy 100.33 31.75) (xy 107.95 31.75)
-		)
-		(stroke
-			(width 0)
-			(type default)
-		)
-	)
-	(wire
-		(pts
-			(xy 100.33 33.02) (xy 100.33 31.75)
-		)
-		(stroke
-			(width 0)
-			(type default)
-		)
-	)
-	(wire
-		(pts
 			(xy 69.85 82.55) (xy 72.39 82.55)
 		)
@@
 	(wire
 		(pts
+			(xy 107.95 34.29) (xy 107.95 38.1)
+		)
+		(stroke
+			(width 0)
+			(type default)
+		)
+	)
+	(wire
+		(pts
 			(xy 48.26 50.8) (xy 48.26 66.04)
 		)
@@
 	(wire
 		(pts
+			(xy 104.14 31.75) (xy 104.14 66.04)
+		)
+		(stroke
+			(width 0)
+			(type default)
+		)
+	)
+	(wire
+		(pts
 			(xy 69.85 85.09) (xy 69.85 82.55)
 		)
@@
 	(wire
 		(pts
+			(xy 99.06 50.8) (xy 99.06 53.34)
+		)
+		(stroke
+			(width 0)
+			(type default)
+		)
+	)
+	(wire
+		(pts
 			(xy 67.31 80.01) (xy 72.39 80.01)
-		)
-		(stroke
-			(width 0)
-			(type default)
-		)
-	)
-	(wire
-		(pts
-			(xy 104.14 34.29) (xy 107.95 34.29)
-		)
-		(stroke
-			(width 0)
-			(type default)
-		)
-	)
-	(wire
-		(pts
-			(xy 104.14 34.29) (xy 104.14 66.04)
 		)
 		(stroke
@@
 	)
 	(symbol
-		(lib_id "power:GND")
-		(at 100.33 48.26 180)
-		(unit 1)
-		(body_style 1)
-		(exclude_from_sim no)
-		(in_bom yes)
-		(on_board yes)
-		(in_pos_files yes)
-		(dnp no)
-		(fields_autoplaced yes)
-		(property "Reference" "#PWR08"
-			(at 100.33 41.91 0)
-			(hide yes)
-			(show_name no)
-			(do_not_autoplace no)
-			(effects
-				(font
-					(size 1.27 1.27)
-				)
-			)
-		)
-		(property "Value" "GND"
-			(at 100.33 43.18 0)
-			(show_name no)
-			(do_not_autoplace no)
-			(effects
-				(font
-					(size 1.27 1.27)
-				)
-			)
-		)
-		(property "Footprint" ""
-			(at 100.33 48.26 0)
-			(hide yes)
-			(show_name no)
-			(do_not_autoplace no)
-			(effects
-				(font
-					(size 1.27 1.27)
-				)
-			)
-		)
-		(property "Datasheet" ""
-			(at 100.33 48.26 0)
-			(hide yes)
-			(show_name no)
-			(do_not_autoplace no)
-			(effects
-				(font
-					(size 1.27 1.27)
-				)
-			)
-		)
-		(property "Description" "Power symbol creates a global label with name \"GND\" , ground"
-			(at 100.33 48.26 0)
-			(hide yes)
-			(show_name no)
-			(do_not_autoplace no)
-			(effects
-				(font
-					(size 1.27 1.27)
-				)
-			)
-		)
-		(pin "1"
-		)
-		(instances
-			(project "Rlaarlo_PDB"
-				(path "/d684c2aa-7b59-4fad-a512-16f34e50dcd7"
-					(reference "#PWR08")
-					(unit 1)
-				)
-			)
-		)
-	)
-	(symbol
 		(lib_id "power:PWR_FLAG")
 		(at 69.85 50.8 0)
@@
 			)
 		)
-		(property "Footprint" "Connector_PinHeader_2.54mm:PinHeader_1x02_P2.54mm_Horizontal"
+		(property "Footprint" "TerminalBlock:TerminalBlock_MaiXu_MX126-5.0-02P_1x02_P5.00mm"
 			(at 125.73 82.55 0)
 			(hide yes)
@@
 	(symbol
 		(lib_id "power:GND")
+		(at 99.06 53.34 0)
+		(unit 1)
+		(body_style 1)
+		(exclude_from_sim no)
+		(in_bom yes)
+		(on_board yes)
+		(in_pos_files yes)
+		(dnp no)
+		(fields_autoplaced yes)
+		(property "Reference" "#PWR010"
+			(at 99.06 59.69 0)
+			(hide yes)
+			(show_name no)
+			(do_not_autoplace no)
+			(effects
+				(font
+					(size 1.27 1.27)
+				)
+			)
+		)
+		(property "Value" "GND"
+			(at 99.06 58.42 0)
+			(show_name no)
+			(do_not_autoplace no)
+			(effects
+				(font
+					(size 1.27 1.27)
+				)
+			)
+		)
+		(property "Footprint" ""
+			(at 99.06 53.34 0)
+			(hide yes)
+			(show_name no)
+			(do_not_autoplace no)
+			(effects
+				(font
+					(size 1.27 1.27)
+				)
+			)
+		)
+		(property "Datasheet" ""
+			(at 99.06 53.34 0)
+			(hide yes)
+			(show_name no)
+			(do_not_autoplace no)
+			(effects
+				(font
+					(size 1.27 1.27)
+				)
+			)
+		)
+		(property "Description" "Power symbol creates a global label with name \"GND\" , ground"
+			(at 99.06 53.34 0)
+			(hide yes)
+			(show_name no)
+			(do_not_autoplace no)
+			(effects
+				(font
+					(size 1.27 1.27)
+				)
+			)
+		)
+		(pin "1"
+		)
+		(instances
+			(project "Rlaarlo_PDB"
+				(path "/d684c2aa-7b59-4fad-a512-16f34e50dcd7"
+					(reference "#PWR010")
+					(unit 1)
+				)
+			)
+		)
+	)
+	(symbol
+		(lib_id "power:GND")
 		(at 107.95 82.55 0)
 		(unit 1)
@@
 	(symbol
 		(lib_id "power:GND")
-		(at 100.33 33.02 0)
+		(at 107.95 38.1 0)
 		(unit 1)
 		(body_style 1)
@@
 		(fields_autoplaced yes)
 		(property "Reference" "#PWR09"
-			(at 100.33 39.37 0)
+			(at 107.95 44.45 0)
 			(hide yes)
 			(show_name no)
@@
 		)
 		(property "Value" "GND"
-			(at 100.33 38.1 0)
+			(at 107.95 43.18 0)
 			(show_name no)
 			(do_not_autoplace no)
@@
 		)
 		(property "Footprint" ""
-			(at 100.33 33.02 0)
-			(hide yes)
-			(show_name no)
-			(do_not_autoplace no)
-			(effects
-				(font
-					(size 1.27 1.27)
-				)
-			)
-		)
-		(property "Datasheet" ""
-			(at 100.33 33.02 0)
+			(at 107.95 38.1 0)
+			(hide yes)
+			(show_name no)
+			(do_not_autoplace no)
+			(effects
+				(font
+					(size 1.27 1.27)
+				)
+			)
+		)
+		(property "Datasheet" ""
+			(at 107.95 38.1 0)
 			(hide yes)
 			(show_name no)
@@
 		)
 		(property "Description" "Power symbol creates a global label with name \"GND\" , ground"
-			(at 100.33 33.02 0)
-			(hide yes)
-			(show_name no)
+			(at 107.95 38.1 0)
+			(hide yes)
+			(show_name no)
