File: acker_pcb/Rlaarlo_PDB/Rlaarlo_PDB.kicad_pcb (KiCad board)
At the start: 2 copper layers, 88.2 x 108.4 mm, 9 parts, among them J1 xt 60, J2 Conn_01x03_Pin, J3 Conn_01x02_Pin, SW1 SW_SPST, SW2 SW_SPST, SW3 SW_SPST

Commit message: pcb updates
Parts:
- added REF**: MountingHole_3.2mm_M3, MountingHole:MountingHole_3.2mm_M3, F.Cu at (154.5, 121.4)
- added REF**: MountingHole_3.2mm_M3, MountingHole:MountingHole_3.2mm_M3, F.Cu at (154.9, 28.6)
- added REF**: MountingHole_3.2mm_M3, MountingHole:MountingHole_3.2mm_M3, F.Cu at (73.7, 28.6)
- added REF**: MountingHole_3.2mm_M3, MountingHole:MountingHole_3.2mm_M3, F.Cu at (73.5, 121.5)
- SW1: value SW_SPST -> SW_SPST_esb
- moved SW3 22.3 mm to (155.0, 100.0), turned to -90 degrees
- moved Buck2 21.7 mm to (134.0, 94.0)
- moved SW2 17.7 mm to (155.0, 79.3), turned to -90 degrees
- moved SW1 17.0 mm to (155.0, 40.0), turned to -90 degrees
- moved J2 9.07 mm to (73.6, 84.4)
- moved J3 7.03 mm to (73.8, 108.0)
- moved Buck1 6.12 mm to (141.2, 132.0)
- moved J1 5.79 mm to (145.0, 61.0)
Routing:
- added copper zone on B.Cu, net GND
- added copper zone on F.Cu, net GND
Other:
- board size 88.2 x 108.4 mm -> 88 x 100 mm

Commit message: pdb updates
Parts:
- jetson v: renamed from J3
- moved SW 13.4 mm to (150.8, 52.8), turned to 180 degrees
- moved SW2 9.72 mm to (150.0, 87.6), turned to 0 degrees
- moved J1 9.50 mm to (143.6, 70.4), turned to 0 degrees
- moved SW3 8.51 mm to (150.0, 106.9), turned to 0 degrees
- renumbered SW1 to SW
Routing:
- net +15V: track 0.00 -> 54.5 mm
- net Net-(J2-Pin_3): track 0.00 -> 34.0 mm
- net Net-(Buck2-v_in_+): track 0.00 -> 25.2 mm
- net Net-(SW1-B): track 0.00 -> 25.0 mm
- net Net-(Buck2-v_out_+): track 0.00 -> 22.4 mm
- net Net-(Buck1-v_in_+): track 0.00 -> 22.2 mm
- net Net-(Buck1-v_out_+): track 0.00 -> 9.09 mm
Other:
- board text added: "Jestson"
- board text added: "SW Jetson"
- board text added: "SW Servo"
- board text added: "SW Vesc"
- board text added: "Servo"
- board text added: "Vesc"

Commit message: final design
Routing:
- net Net-(Buck1-v_out_+): track 9.09 -> 14.2 mm
- net Net-(Buck1-v_in_+): track 22.2 -> 21.1 mm
Changed lines of the file:
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@@
 		(capping no)
 		(filling no)
+		(zone_defaults)
 		(pcbplotparams
 			(layerselection 0x00000000_00000000_55555555_5755f5ff)
 			(plot_on_all_layers_selection 0x00000000_00000000_00000000_00000000)
 			(disableapertmacros no)
-			(usegerberextensions no)
+			(usegerberextensions yes)
 			(usegerberattributes yes)
 			(usegerberadvancedattributes yes)
-			(creategerberjobfile yes)
+			(creategerberjobfile no)
 			(dashed_line_dash_ratio 12)
 			(dashed_line_gap_ratio 3)
@@
 			(outputformat 1)
 			(mirror no)
-			(drillshape 1)
+			(drillshape 0)
 			(scaleselection 1)
 			(outputdirectory "")
@@
 		(duplicate_pad_numbers_are_jumpers no)
 		(pad "1" thru_hole circle
+			(at 29 -3 90)
+			(size 1.7 1.7)
+			(drill 1)
+			(layers "*.Cu" "*.Mask")
+			(remove_unused_layers no)
+			(net "Net-(Buck1-v_in_+)")
+			(pinfunction "v_in_+_1")
+			(pintype "power_in")
+		)
+		(pad "2" thru_hole circle
 			(at 15 -3 90)
 			(size 1.7 1.7)
@@
 			(layers "*.Cu" "*.Mask")
 			(remove_unused_layers no)
-			(net "Net-(Buck1-v_in_+)")
-			(pinfunction "v_in_+_1")
-			(pintype "power_in")
-		)
-		(pad "2" thru_hole circle
-			(at 29 -3 90)
-			(size 1.7 1.7)
-			(drill 1)
-			(layers "*.Cu" "*.Mask")
-			(remove_unused_layers no)
 			(net "GND")
 			(pinfunction "v_in_-_2")
@@
 		)
 		(pad "3" thru_hole circle
-			(at 15 -60 90)
+			(at 29 -60 90)
 			(size 1.7 1.7)
 			(drill 1)
@@
 		)
 		(pad "4" thru_hole circle
-			(at 29 -60 90)
+			(at 15 -60 90)
 			(size 1.7 1.7)
 			(drill 1)
@@
 		(attr through_hole)
 		(duplicate_pad_numbers_are_jumpers no)
-		(fp_line
-			(start -3.09 -4.09)
-			(end 7.65 -4.09)
-			(stroke
-				(width 0.12)
-				(type solid)
-			)
-			(layer "F.SilkS")
-		)
-		(fp_line
-			(start -3.09 3.95)
-			(end -3.09 -4.09)
-			(stroke
-				(width 0.12)
-				(type solid)
-			)
-			(layer "F.SilkS")
-		)
-		(fp_line
-			(start -0.27 3.95)
-			(end -3.09 3.95)
-			(stroke
-				(width 0.12)
-				(type solid)
-			)
-			(layer "F.SilkS")
-		)
-		(fp_line
-			(start 7.65 -4.09)
-			(end 7.65 3.95)
-			(stroke
-				(width 0.12)
-				(type solid)
-			)
-			(layer "F.SilkS")
-		)
-		(fp_line
-			(start 7.65 3.95)
-			(end 0.33 3.95)
-			(stroke
-				(width 0.12)
-				(type solid)
-			)
-			(layer "F.SilkS")
-		)
 		(fp_rect
 			(start -3.97 -8.47)
@@
 		)
 		(fp_line
-			(start -2.97 -3.97)
-			(end 7.53 -3.97)
-			(stroke
-				(width 0.1)
-				(type solid)
-			)
-			(layer "F.Fab")
-		)
-		(fp_line
-			(start -2.97 1.88)
-			(end -2.97 -3.97)
-			(stroke
-				(width 0.1)
-				(type solid)
-			)
-			(layer "F.Fab")
-		)
-		(fp_line
-			(start -1.02 3.83)
-			(end -2.97 1.88)
-			(stroke
-				(width 0.1)
-				(type solid)
-			)
-			(layer "F.Fab")
-		)
-		(fp_line
 			(start 1.048 -1.183)
 			(end -1.183 1.048)
@@
 			(start 6.243 -0.988)
 			(end 4.012 1.243)
-			(stroke
-				(width 0.1)
-				(type solid)
-			)
-			(layer "F.Fab")
-		)
-		(fp_line
-			(start 7.53 -3.97)
-			(end 7.53 3.83)
-			(stroke
-				(width 0.1)
-				(type solid)
-			)
-			(layer "F.Fab")
-		)
-		(fp_line
-			(start 7.53 3.83)
-			(end -1.02 3.83)
 			(stroke
 				(width 0.1)
@@
 		(attr through_hole)
 		(duplicate_pad_numbers_are_jumpers no)
-		(fp_line
-			(start -2.88 -3.87)
-			(end 7.86 -3.87)
-			(stroke
-				(width 0.12)
-				(type solid)
-			)
-			(layer "F.SilkS")
-		)
-		(fp_line
-			(start -2.88 4.17)
-			(end -2.88 -3.87)
-			(stroke
-				(width 0.12)
-				(type solid)
-			)
-			(layer "F.SilkS")
-		)
-		(fp_line
-			(start -0.06 4.17)
-			(end -2.88 4.17)
-			(stroke
-				(width 0.12)
-				(type solid)
-			)
-			(layer "F.SilkS")
-		)
-		(fp_line
-			(start 7.86 -3.87)
-			(end 7.86 4.17)
-			(stroke
-				(width 0.12)
-				(type solid)
-			)
-			(layer "F.SilkS")
-		)
-		(fp_line
-			(start 7.86 4.17)
-			(end 0.54 4.17)
-			(stroke
-				(width 0.12)
-				(type solid)
-			)
-			(layer "F.SilkS")
-		)
 		(fp_rect
 			(start -3.76 -8.25)
@@
 		)
 		(fp_line
-			(start -2.76 -3.75)
-			(end 7.74 -3.75)
-			(stroke
-				(width 0.1)
-				(type solid)
-			)
-			(layer "F.Fab")
-		)
-		(fp_line
-			(start -2.76 2.1)
-			(end -2.76 -3.75)
-			(stroke
-				(width 0.1)
-				(type solid)
-			)
-			(layer "F.Fab")
-		)
-		(fp_line
-			(start -0.81 4.05)
-			(end -2.76 2.1)
-			(stroke
-				(width 0.1)
-				(type solid)
-			)
-			(layer "F.Fab")
-		)
-		(fp_line
 			(start 1.258 -0.963)
 			(end -0.973 1.268)
@@
 			(start 6.453 -0.768)
 			(end 4.222 1.463)
-			(stroke
-				(width 0.1)
-				(type solid)
-			)
-			(layer "F.Fab")
-		)
-		(fp_line
-			(start 7.74 -3.75)
-			(end 7.74 4.05)
-			(stroke
-				(width 0.1)
-				(type solid)
-			)
-			(layer "F.Fab")
-		)
-		(fp_line
-			(start 7.74 4.05)
-			(end -0.81 4.05)
 			(stroke
 				(width 0.1)
@@
 	)
 	(segment
-		(start 81.2 116.97)
-		(end 77.78 116.97)
-		(width 3)
-		(layer "F.Cu")
-		(net "Net-(Buck1-v_out_+)")
-	)
-	(segment
-		(start 77.78 116.97)
+		(start 75.749898 112.96)
 		(end 73.77 112.96)
 		(width 3)
@@
 	)
 	(segment
-		(start 146.952398 116.97)
-		(end 138.2 116.97)
+		(start 81.2 107.509898)
+		(end 75.749898 112.96)
 		(width 3)
 		(layer "F.Cu")
+		(net "Net-(Buck1-v_out_+)")
+	)
+	(segment
+		(start 81.2 102.97)
+		(end 81.2 107.509898)
+		(width 3)
+		(layer "F.Cu")
+		(net "Net-(Buck1-v_out_+)")
+	)
+	(segment
+		(start 155.03 106.977144)
+		(end 151.994644 110.0125)
+		(width 3)
+		(layer "B.Cu")
+		(net "Net-(Buck1-v_in_+)")
+	)
+	(segment
+		(start 151.994644 110.0125)
+		(end 145.2425 110.0125)
+		(width 3)
+		(layer "B.Cu")
 		(net "Net-(Buck1-v_in_+)")
 	)
 	(segment
 		(start 155.03 106.9125)
-		(end 155.03 108.892398)
+		(end 155.03 106.977144)
 		(width 3)
-		(layer "F.Cu")
+		(layer "B.Cu")
 		(net "Net-(Buck1-v_in_+)")
 	)
 	(segment
-		(start 155.03 108.892398)
-		(end 146.952398 116.97)
+		(start 145.2425 110.0125)
+		(end 138.2 102.97)
 		(width 3)
-		(layer "F.Cu")
+		(layer "B.Cu")
 		(net "Net-(Buck1-v_in_+)")
 	)
